Commit message: Update

File: robot/src/scara_robot/urdf/scara.urdf.xacro (robot description, xacro)
@@ -1,15 +1,15 @@
 <?xml version="1.0"?>
 <robot name="scara">
-    <material name="red">
-        <color rgba="1.0 0 0 1.0"/>
+    <material name="yellow">
+        <color rgba="1.0 1.0 0 1.0"/>
+    </material>
+    <material name="black">
+        <color rgba="0 0 0 1.0"/>
     </material>
     <material name="green">
         <color rgba="0 1.0 0 1.0"/>
     </material>
-    <material name="blue">
-        <color rgba="0 0 1.0 1.0"/>
-    </material>
-    <material name="white">
-        <color rgba="1.0 1.0 1.0 1.0"/>
+    <material name="pink">
+        <color rgba="1.0 0 1.0 1.0"/>
     </material>
     <!-- base link -->
@@ -20,5 +20,5 @@
                 <box size="0.2 0.4 0.6"/>
             </geometry>
-            <material name="white"/>
+            <material name="pink"/>
         </visual>
     </link>
@@ -30,5 +30,5 @@
                 <box size="0.2 0.6 0.1"/>
             </geometry>
-            <material name="blue"/>
+            <material name="green"/>
         </visual>
     </link>
@@ -48,5 +48,5 @@
                 <box size="0.2 0.6 0.3"/>
             </geometry>
-            <material name="green"/>
+            <material name="black"/>
         </visual>
     </link>
@@ -66,5 +66,5 @@
                 <cylinder length="1" radius="0.01"/>
             </geometry>
-            <material name="red"/>
+            <material name="yellow"/>
         </visual>
     </link>
